File: Keyboard/SpyderDumbKeyboard.kicad_sch (KiCad schematic)
At the start: 6 parts, among them J1 KeyboardOutput, J2 KeyboardOutput, U2 STM32F030R8Tx

Commit message: Fixed minor issues & plotted gerber
Parts:
- removed U2: STM32F030R8Tx, Package_QFP:LQFP-64_10x10mm_P0.5mm, symbol MCU_ST_STM32F0:STM32F030R8Tx
- added D37: LED_Small, LED_SMD:LED_0603_1608Metric_Pad1.05x0.95mm_HandSolder, symbol Device:LED_Small
- added R2, R3, R4, R5, R6, R7: 10kΩ, Resistor_SMD:R_0603_1608Metric_Pad0.98x0.95mm_HandSolder, symbol Device:R_Small
- added R8: R_Small, Resistor_SMD:R_0603_1608Metric_Pad0.98x0.95mm_HandSolder, symbol Device:R_Small
- added U1: STM32G030K8Tx, Package_QFP:LQFP-32_7x7mm_P0.8mm, symbol MCU_ST_STM32G0:STM32G030K8Tx
- C1, C2: footprint (none) -> Capacitor_SMD:C_0603_1608Metric_Pad1.08x0.95mm_HandSolder
- J1: footprint (none) -> Connector_PinHeader_2.54mm:PinHeader_1x05_P2.54mm_Vertical
- J2: value KeyboardOutput -> Programmer; footprint (none) -> Connector_PinHeader_2.54mm:PinHeader_1x05_P2.54mm_Vertical
- R1: footprint (none) -> Resistor_SMD:R_0603_1608Metric_Pad0.98x0.95mm_HandSolder
Connections:
- net +3V3: now also U1.4 (VDD)
- net CS: now also U1.11 (PA4)
- net GND: now also R1.2, R2.2, R3.2, R4.2, R5.2, R6.2, R7.2, R8.1, U1.5 (VSS); no longer R1.1
- net MISO: now also U1.13 (PA6)
- net RESET: now also U1.6 (NRST)
- net SCLK: now also U1.12 (PA5)
- net SWCLK: now also R7.1, U1.25 (PA14)
- net SWDIO: now also U1.24 (PA13)
- new net: D37.2 (A), U1.9 (PA2)
- new net: D37.1 (K), R8.2
- new net c0: R1.1, U1.30 (PB6)
- new net c1: R2.1, U1.31 (PB7)
- new net c2: R3.1, U1.8 (PA1)
- new net c3: R4.1, U1.1 (PB9)
- new net c4: R5.1, U1.32 (PB8)
- new net c5: R6.1, U1.7 (PA0)
- new net r0: U1.15 (PB0)
- new net r1: U1.16 (PB1)
- new net r2: U1.17 (PB2)
- new net r3: U1.27 (PB3)
- new net r4: U1.28 (PB4)
- new net r5: U1.29 (PB5)
- no-connect marks 0 -> 9
Other:
- sheet keyboard ports: added col0, col1, col2, col3, col4, col5, row0, row1, row2, row3, row4, row5; removed none
