File: mainBoard/mainBoard.kicad_pcb (KiCad board)
At the start: 4 copper layers, 53.3 x 50 mm, 30 parts, among them J1 Battery Output, J2 Conn_01x06_Pin, J3 Keyboard, J4 display, J5 RYLR998, M1 Vibration Motor, Q1 IRLML2502, U1 STM32G030K8Tx, U2 AMS1117-3.3, U3 W25Q128JVS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

Commit message: Added Graphics
Added version, creators, board name, and funny qr code.
Routing:
- net /BL: track 65.3 -> 70.9 mm
- net /displayRESET: track 59.1 -> 64.5 mm
- net /DC: track 66.4 -> 70.8 mm
Other:
- board text added: "+5V"
- board text added: "By: Luke & Colin"
- board text added: "DISPLAY"
- board text added: "GND CS SCK MISO 3V3"
- board text added: "MAINBOARD"
- board text added: "POWER"
- board text added: "RYLR998"
- board text added: "Spyder v2"
- board text removed: "5V"

Commit message: Fixed Minor Issue
Parts:
- removed C4, C5: 22pF, Capacitor_SMD:C_0603_1608Metric_Pad1.08x0.95mm_HandSolder
- removed Y1: 48MHz, Crystal:Crystal_HC49-U_Vertical
Connections:
- U1 pad 2: Net-(U1-PC14) -> unconnected-(U1-PC14-Pad2)
- U1 pad 3: Net-(U1-PC15) -> unconnected-(U1-PC15-Pad3)
Routing:
- net Net-(U1-PC14): track 13.9 -> 0.00 mm
- net Net-(U1-PC15): track 13.8 -> 0.00 mm
- net GND: track 24.7 -> 22.7 mm, vias 10 -> 9

Commit message: Fixed minor issues & plotted gerber
Parts:
- added D2: Indicator LED, LED_SMD:LED_0603_1608Metric_Pad1.05x0.95mm_HandSolder, F.Cu at (138.6, 45.4)
- added R4: 10kΩ, Resistor_SMD:R_0603_1608Metric_Pad0.98x0.95mm_HandSolder, F.Cu at (125.7, 42.5)
- added R5: 100Ω, Resistor_SMD:R_0603_1608Metric_Pad0.98x0.95mm_HandSolder, F.Cu at (138.4, 40.8)
Connections:
- U1 pad 14: unconnected-(U1-PA7-Pad14) -> Net-(D2-A)
Routing:
- net Net-(D2-A): track 0.00 -> 3.93 mm
- net Net-(D2-K): track 0.00 -> 2.90 mm
- net GND: track 22.7 -> 24.0 mm, vias 9 -> 11
